File: project_01/KICAD/EDES301NOTER/HallSwitch.kicad_sch (KiCad schematic)
At the start: 8 parts, among them Q6 BSS84, U2 DRV5032FCDBZR

Commit message: Revise Boost5V schematic and add STIKE symbols
Refactor Boost5V.kicad_sch: updated title block and paper size, reorganized and renamed many symbol definitions (capacitor/inductor/diode/resistor/LED/driver), adjusted pin assignments, footprints, datasheet links and symbol graphics. Added new STIKE-related schematic symbols (Slide Switch, LipoConnection) and multiple KiCad footprint/symbol files under KICAD Files. Added project backup zips and freerouting.dsn, removed a temporary .kicad_sch.lck, and updated project metadata files (.kicad_pcb, .kicad_prl, .kicad_pro, .kicad_sch).
Parts:
- removed C12, C13: 1uF, Footprints:CAPC1608X90N, symbol Device:C
- removed D1: B0530W-7-F, B0530W-7-F:SOD3715X145N, symbol B0530W-7-F:B0530W-7-F
- removed Q6: BSS84, Package_TO_SOT_SMD:SOT-23, symbol Transistor_FET:BSS84
- removed R14: 10k, Footprints:RESC1607X60N, symbol Device:R
- removed R15, R16: 100k, Footprints:RESC1607X60N, symbol Device:R
- removed U2: DRV5032FCDBZR, DRV5032FCDBZR:DBZ0003A-IPC_A, symbol DRV5032FCDBZR:DRV5032FCDBZR
Other:
- title: Hall Effect Power Switch -> ePaper Support Circuitry
