File: project_01/KICAD/EDES301NOTER/TFTDisp.kicad_sch (KiCad schematic)
At the start: 12 parts, among them Q1 S8050, Q3 BSS84

Commit message: Revise Boost5V schematic and add STIKE symbols
Refactor Boost5V.kicad_sch: updated title block and paper size, reorganized and renamed many symbol definitions (capacitor/inductor/diode/resistor/LED/driver), adjusted pin assignments, footprints, datasheet links and symbol graphics. Added new STIKE-related schematic symbols (Slide Switch, LipoConnection) and multiple KiCad footprint/symbol files under KICAD Files. Added project backup zips and freerouting.dsn, removed a temporary .kicad_sch.lck, and updated project metadata files (.kicad_pcb, .kicad_prl, .kicad_pro, .kicad_sch).
Parts:
- removed C5: 0.1uF, Footprints:CAPC1608X90, symbol Device:C
- removed C7: 1uF, Footprints:CAPC1608X90N, symbol Device:C
- removed Q1: S8050, Package_TO_SOT_THT:TO-92_Inline, symbol Transistor_BJT:S8050
- removed Q3: BSS84, Package_TO_SOT_SMD:SOT-23, symbol Transistor_FET:BSS84
- removed R1, R2, R3, R4: 10R, Footprints:RESC2012X60N, symbol Device:R
- removed R5, R6: 1K, Footprints:RESC1607X60N, symbol Device:R
- removed R8: 100k, Footprints:RESC1607X60N, symbol Device:R
- removed U5: ~, FH34SRJ-18S-0.5SH:CONN18x1_FH34SRJ-18S-0.5SH50_HIR, symbol YT280S010:DISPLAY
Other:
- note removed: "(NO)Low Power Switch"
- title: TFT Display Connection Circuitry -> ePaper Support Circuitry
