File: project_01/KICAD/EDES301NOTER/ePaperSupport.kicad_sch (KiCad schematic)
At the start: 21 parts, among them J1 FH12-24S-0.5SH55, Q4 BSS84, U7 PMF250XNEX

Commit message: Revise Boost5V schematic and add STIKE symbols
Refactor Boost5V.kicad_sch: updated title block and paper size, reorganized and renamed many symbol definitions (capacitor/inductor/diode/resistor/LED/driver), adjusted pin assignments, footprints, datasheet links and symbol graphics. Added new STIKE-related schematic symbols (Slide Switch, LipoConnection) and multiple KiCad footprint/symbol files under KICAD Files. Added project backup zips and freerouting.dsn, removed a temporary .kicad_sch.lck, and updated project metadata files (.kicad_pcb, .kicad_prl, .kicad_pro, .kicad_sch).
Parts:
- removed C14, C16, C17, C19, C20, C21, C22, C9: 1uF, Footprints:CAPC1608X90N, symbol Device:C
- removed C15, C18: 4.7uF, Footprints:CAPC1608X90N, symbol Device:C
- removed C6: 0.1uF, Footprints:CAPC1608X90, symbol Device:C
- removed D2, D3, D4: B0530W-7-F, B0530W-7-F:SOD3715X145N, symbol B0530W-7-F:B0530W-7-F
- removed J1: FH12-24S-0.5SH55, CF4224FH0R0-05-NH:CONN24X1_FH12-24S-0.5SH55_HIR, symbol CF4224FH0R0-05-NH:FH12-24S-0.5SH55
- removed L2: 47uH, IFSC2020DEER470M01:IND_IFSC-2020DE-01_VIS, symbol IFSC2020DEER470M01:IFSC2020DEER470M01
- removed Q4: BSS84, Package_TO_SOT_SMD:SOT-23, symbol Transistor_FET:BSS84
- removed R17: 1M, Footprints:RESC1607X60N, symbol Device:R
- removed R18: 2.2, Footprints:RESC1607X60N, symbol Device:R
- removed R9: 100k, Footprints:RESC1607X60N, symbol Device:R
- removed U7: PMF250XNEX, PMF250XNEX:PMF250XNEX_NEX, symbol PMF250XNEX:PMF250XNEX
Connections:
- no-connect marks 5 -> 0
Other:
- note removed: "(NO)Low Power Switch"
