File: project_01/KICAD/ProjectBackup6AM/ProjectBackup6AM.kicad_sch (KiCad schematic)
At the start: 6 parts, among them SW1 Boot, SW2 RST

Commit message: Update KiCad schematics to v10; clean backups
Bump KiCad schematic version/generator to v10 and normalize symbol/property metadata in Boost5V.kicad_sch (add show_name/do_not_autoplace/hide/in_pos_files, standardize pin names/numbers/types and orientations). Apply similar component property adjustments (e.g. TPB4056, XC6206, TPS613222) and update related project PCB/PRO/PRL/SCH files. Add ProjectBackupFINAL and several new zip backups, and remove many old backup, cache and lock files to clean up the repository. These are primarily metadata and housekeeping changes, not functional circuit edits.
Parts:
- U4, U7, U8: value ~ -> (none)
Connections:
- net ESP32-S3-N16R8/LCD_SCK: no longer U8.3 (LCD_SCK)
- net ESP32-S3-N16R8/RST: now also SW2.3; no longer SW2.1
- net GND: now also SW2.1; no longer SW2.3
Other:
- moved on the sheet: U7, U8
