File: project_01/KICAD/ProjectBackup6AM/STIKE-ESP32.kicad_sch (KiCad schematic)
At the start: 1 part, among them U6 ESP32-S3-WROOM-1-N16R8

Commit message: Update KiCad schematics to v10; clean backups
Bump KiCad schematic version/generator to v10 and normalize symbol/property metadata in Boost5V.kicad_sch (add show_name/do_not_autoplace/hide/in_pos_files, standardize pin names/numbers/types and orientations). Apply similar component property adjustments (e.g. TPB4056, XC6206, TPS613222) and update related project PCB/PRO/PRL/SCH files. Add ProjectBackupFINAL and several new zip backups, and remove many old backup, cache and lock files to clean up the repository. These are primarily metadata and housekeeping changes, not functional circuit edits.
Connections:
- net EP_BUSY: now also U6.10 (IO17); no longer U6.4 (IO4)
